Commit message: Add gripper only taskmap. Set seven points for pose tracking

File: src/fabrics_sim/models/robots/urdf/cs63_tesollo/cs63_tesollo.urdf (robot description, URDF)
Before this commit: robot cs63_tesollo, 25 links, 24 joints
Links:
- added link palm_x
- added link palm_x_neg
- added link palm_y
- added link palm_y_neg
- added link palm_z
- added link palm_z_neg
- added link tip1_force_frame
- added link tip2_force_frame
- added link tip3_force_frame
Joints:
- added joint palm_x_joint: type fixed, parent palm_link, child palm_x, origin xyz=0.25 0.0 0.0 rpy=0 0 0
- added joint palm_x_neg_joint: type fixed, parent palm_link, child palm_x_neg, origin xyz=-0.25 0.0 0.0 rpy=0 0 0
- added joint palm_y_joint: type fixed, parent palm_link, child palm_y, origin xyz=0.0 0.25 0.0 rpy=0 0 0
- added joint palm_y_neg_joint: type fixed, parent palm_link, child palm_y_neg, origin xyz=0.0 -0.25 0.0 rpy=0 0 0
- added joint palm_z_joint: type fixed, parent palm_link, child palm_z, origin xyz=0.0 0.0 0.25 rpy=0 0 0
- added joint palm_z_neg_joint: type fixed, parent palm_link, child palm_z_neg, origin xyz=0.0 0.0 -0.25 rpy=0 0 0
- added joint tip1_force_frame_joint: type fixed, parent F1_TIP, child tip1_force_frame, origin xyz=0.045 0.0 0.0 rpy=0 0 0
- added joint tip2_force_frame_joint: type fixed, parent F2_TIP, child tip2_force_frame, origin xyz=0.045 0.0 0.0 rpy=0 0 0
- added joint tip3_force_frame_joint: type fixed, parent F3_TIP, child tip3_force_frame, origin xyz=0.045 0.0 0.0 rpy=0 0 0

Commit message: offset from 0.25 to 0.10

File: src/fabrics_sim/models/robots/urdf/cs63_tesollo/cs63_tesollo.urdf (robot description, URDF)
Before this commit: robot cs63_tesollo, 34 links, 33 joints
Joints:
- joint palm_x_joint: origin xyz=0.25 0.0 0.0 rpy=0 0 0 -> xyz=0.1 0.0 0.0 rpy=0 0 0
- joint palm_x_neg_joint: origin xyz=-0.25 0.0 0.0 rpy=0 0 0 -> xyz=-0.1 0.0 0.0 rpy=0 0 0
- joint palm_y_joint: origin xyz=0.0 0.25 0.0 rpy=0 0 0 -> xyz=0.0 0.1 0.0 rpy=0 0 0
- joint palm_y_neg_joint: origin xyz=0.0 -0.25 0.0 rpy=0 0 0 -> xyz=0.0 -0.1 0.0 rpy=0 0 0
- joint palm_z_joint: origin xyz=0.0 0.0 0.25 rpy=0 0 0 -> xyz=0.0 0.0 0.1 rpy=0 0 0
- joint palm_z_neg_joint: origin xyz=0.0 0.0 -0.25 rpy=0 0 0 -> xyz=0.0 0.0 -0.1 rpy=0 0 0
